File: blake-intro/blake-intro.sch (KiCad schematic (older format))
At the start: 2 parts

Commit message: schematic finished
Parts:
- removed D?: LED, symbol Device:LED
- added BT1, BT2: 3V, Battery:BatteryHolder_LINX_BAT-HLD-012-SMT, symbol Device:Battery_Cell
- added C1: 0.01u, Capacitor_SMD:C_0805_2012Metric, symbol Device:C
- added C2: 10u, Capacitor_SMD:C_0805_2012Metric, symbol Device:C
- added D1: LED, LED_SMD:LED_0805_2012Metric, symbol Device:LED
- added R1: 5k, Resistor_SMD:R_0805_2012Metric, symbol Device:R
- added R2: 10k, Resistor_SMD:R_0805_2012Metric, symbol Device:R
- gave numbers to parts that had none: 1
Connections:
- net GND: now reaches U1.1 (GND)
- net GND: now also BT2.2 (-), C1.2, C2.2, D1.1 (K)
- net at U1.2 (TR): now also U1.6 (THR), C2.1, R2.2
- net at U1.3 (Q): now also D1.2 (A)
- net VCC: now reaches U1.4 (R)
- net VCC: now also U1.8 (VCC), BT1.1 (+), R1.1
- net at U1.5 (CV): now also C1.1
- net at U1.7 (DIS): now also R1.2, R2.1
- new net: BT1.2 (-), BT2.1 (+)
Other:
- moved on the sheet: U1
