File: TomasMendoza/TomasMendoza.sch (KiCad schematic (older format))
At the start: 2 parts

Commit message: This is my intro project
Parts:
- added BT1, BT2, BT3: 3V, Battery:BatteryHolder_LINX_BAT-HLD-012-SMT, symbol Device:Battery_Cell
- added C1: 10*10^(-6) F, Capacitor_SMD:C_0805_2012Metric, symbol Device:C
- added C2: 0.01*10^(-6) F, Capacitor_SMD:C_0805_2012Metric, symbol Device:C
- added R1: 10k ohms, Resistor_SMD:R_0805_2012Metric, symbol Device:R
- added R2: 5k ohms, Resistor_SMD:R_0805_2012Metric, symbol Device:R
- D1: renamed from D?; footprint (none) -> LED_SMD:LED_0805_2012Metric
- gave numbers to parts that had none: 1
Connections:
- net GND: now reaches U1.1 (GND)
- net GND: now also D1.1 (K), U1.2 (TR), U1.4 (R), U1.6 (THR), U1.8 (VCC), BT1.1 (+), BT3.2 (-), C1.1, C1.2, C2.2, R1.1, R2.2
- net at D1.2 (A), U1.3 (Q): now also U1.7 (DIS), R1.2, R2.1
- net at U1.5 (CV): now also C2.1
- new net: BT1.2 (-), BT2.1 (+)
- new net: BT2.2 (-), BT3.1 (+)
Changed lines of the file:
@@
 $EndDescr
 $Comp
-L Timer:LM555xM U?
+L Device:R R1
+U 1 1 61537EC9
+P 4350 3350
+F 0 "R1" H 4420 3396 50  0000 L CNN
+F 1 "10k ohms" H 4420 3305 50  0000 L CNN
+F 2 "Resistor_SMD:R_0805_2012Metric" V 4280 3350 50  0001 C CNN
+F 3 "~" H 4350 3350 50  0001 C CNN
+	1    4350 3350
+	1    0    0    -1
+$EndComp
+$Comp
+L Device:R R2
+U 1 1 61539B37
+P 4350 3850
+F 0 "R2" H 4420 3896 50  0000 L CNN
+F 1 "5k ohms" H 4420 3805 50  0000 L CNN
+F 2 "Resistor_SMD:R_0805_2012Metric" V 4280 3850 50  0001 C CNN
+F 3 "~" H 4350 3850 50  0001 C CNN
+	1    4350 3850
+	1    0    0    -1
+$EndComp
+Connection ~ 5700 4850
+$Comp
+L Device:C C2
+U 1 1 6153CF6F
+P 4900 4650
+F 0 "C2" H 5015 4696 50  0000 L CNN
+F 1 "0.01*10^(-6) F" H 5015 4605 50  0000 L CNN
+F 2 "Capacitor_SMD:C_0805_2012Metric" H 4938 4500 50  0001 C CNN
+F 3 "~" H 4900 4650 50  0001 C CNN
+	1    4900 4650
+	1    0    0    -1
+$EndComp
+Wire Wire Line
+	6750 3950 6750 3400
+Wire Wire Line
+	7050 3400 7050 4850
+$Comp
+L Device:LED D1
+U 1 1 614CF25E
+P 6900 3400
+F 0 "D1" H 6893 3145 50  0000 C CNN
+F 1 "LED" H 6893 3236 50  0000 C CNN
+F 2 "LED_SMD:LED_0805_2012Metric" H 6900 3400 50  0001 C CNN
+F 3 "~" H 6900 3400 50  0001 C CNN
+	1    6900 3400
+	-1   0    0    1
+$EndComp
+$Comp
+L power:VCC #PWR01
+U 1 1 61542BC1
+P 5700 2350
+F 0 "#PWR01" H 5700 2200 50  0001 C CNN
+F 1 "VCC" H 5715 2523 50  0000 C CNN
+F 2 "" H 5700 2350 50  0001 C CNN
+F 3 "" H 5700 2350 50  0001 C CNN
+	1    5700 2350
+	1    0    0    -1
+$EndComp
+Wire Wire Line
+	4900 4500 4900 4150
+Wire Wire Line
+	4900 4800 4900 4850
+$Comp
+L Device:C C1
+U 1 1 6153DF91
+P 4350 4700
+F 0 "C1" H 4465 4746 50  0000 L CNN
+F 1 "10*10^(-6) F" H 4465 4655 50  0000 L CNN
+F 2 "Capacitor_SMD:C_0805_2012Metric" H 4388 4550 50  0001 C CNN
+F 3 "~" H 4350 4700 50  0001 C CNN
+	1    4350 4700
+	1    0    0    -1
+$EndComp
+Wire Wire Line
+	4350 3700 6200 3700
+Wire Wire Line
+	4350 4850 4900 4850
+Connection ~ 4900 4850
+Wire Wire Line
+	4350 3700 4350 3500
+Connection ~ 4350 3700
+Wire Wire Line
+	4350 3200 4350 2350
+Wire Wire Line
+	4350 2350 5700 2350
+Connection ~ 5700 2350
+Wire Wire Line
+	5200 2700 6450 2700
+Wire Wire Line
+	6450 2700 6450 4350
+Wire Wire Line
+	3150 2100 5700 2100
+Wire Wire Line
+	5700 2100 5700 2350
+Wire Wire Line
+	3150 2800 3150 2100
+Wire Wire Line
+	3150 4050 3150 3650
+$Comp
+L Device:Battery_Cell BT3
+U 1 1 6153F8E5
+P 3150 4250
+F 0 "BT3" H 3268 4346 50  0000 L CNN
+F 1 "3V" H 3268 4255 50  0000 L CNN
+F 2 "Battery:BatteryHolder_LINX_BAT-HLD-012-SMT" V 3150 4310 50  0001 C CNN
+F 3 "~" V 3150 4310 50  0001 C CNN
+	1    3150 4250
+	1    0    0    -1
+$EndComp
+$Comp
+L Device:Battery_Cell BT2
+U 1 1 6153F537
+P 3150 3550
+F 0 "BT2" H 3268 3646 50  0000 L CNN
+F 1 "3V" H 3268 3555 50  0000 L CNN
+F 2 "Battery:BatteryHolder_LINX_BAT-HLD-012-SMT" V 3150 3610 50  0001 C CNN
+F 3 "~" V 3150 3610 50  0001 C CNN
+	1    3150 3550
+	1    0    0    -1
+$EndComp
+Wire Wire Line
+	3150 3350 3150 3100
+$Comp
+L Device:Battery_Cell BT1
+U 1 1 6153EB74
+P 3150 3000
+F 0 "BT1" H 3268 3096 50  0000 L CNN
+F 1 "3V" H 3268 3005 50  0000 L CNN
+F 2 "Battery:BatteryHolder_LINX_BAT-HLD-012-SMT" V 3150 3060 50  0001 C CNN
+F 3 "~" V 3150 3060 50  0001 C CNN
+	1    3150 3000
+	1    0    0    -1
+$EndComp
+Wire Wire Line
+	7050 4850 5700 4850
+Wire Wire Line
+	4900 4150 5200 4150
+Wire Wire Line
+	6200 3950 6750 3950
+Wire Wire Line
+	6200 3700 6200 3950
+Connection ~ 6200 3950
+Wire Wire Line
+	6200 3950 6200 4150
+Wire Wire Line
+	5200 3950 5200 2700
+Wire Wire Line
+	5700 4550 5700 4850
+$Comp
+L Timer:LM555xM U1
 U 1 1 614CCCEE
 P 5700 4150
-F 0 "U?" H 5700 4731 50  0000 C CNN
+F 0 "U1" H 5700 4731 50  0000 C CNN
 F 1 "LM555xM" H 5700 4640 50  0000 C CNN
 F 2 "Package_SO:SOIC-8_3.9x4.9mm_P1.27mm" H 6550 3750 50  0001 C CNN
@@
 	1    0    0    -1
 $EndComp
-$Comp
-L Device:LED D?
-U 1 1 614CF25E
-P 6900 3400
-F 0 "D?" H 6893 3145 50  0000 C CNN
-F 1 "LED" H 6893 3236 50  0000 C CNN
-F 2 "" H 6900 3400 50  0001 C CNN
-F 3 "~" H 6900 3400 50  0001 C CNN
-	1    6900 3400
-	-1   0    0    1
-$EndComp
-Wire Wire Line
-	6200 3950 6750 3950
-Wire Wire Line
-	6750 3950 6750 3400
+Wire Wire Line
+	5200 4350 4850 4350
+Wire Wire Line
+	4850 4350 4850 3750
+Wire Wire Line
+	4850 3750 5700 3750
+Connection ~ 5700 3750
+Wire Wire Line
+	6200 6250 3750 6250
+Wire Wire Line
+	3750 4200 4350 4200
+Wire Wire Line
+	3750 4200 3750 6250
+Wire Wire Line
+	4350 4000 4350 4200
+Wire Wire Line
+	4350 4200 4350 4550
+Connection ~ 4350 4200
+Wire Wire Line
+	4900 4850 5700 4850
+Connection ~ 6200 4350
+Wire Wire Line
+	6200 4350 6450 4350
+Wire Wire Line
+	6200 4350 6200 6250
+Wire Wire Line
+	3150 6250 3750 6250
+Connection ~ 3750 6250
+Wire Wire Line
+	3150 4350 3150 4550
+Connection ~ 5700 4550
+$Comp
+L power:GND #PWR02
+U 1 1 6153AF7B
+P 5700 5300
+F 0 "#PWR02" H 5700 5050 50  0001 C CNN
+F 1 "GND" H 5705 5127 50  0000 C CNN
+F 2 "" H 5700 5300 50  0001 C CNN
+F 3 "" H 5700 5300 50  0001 C CNN
+	1    5700 5300
+	1    0    0    -1
+$EndComp
+Wire Wire Line
+	9000 5750 5700 5750
+Wire Wire Line
+	5700 4850 5700 5300
+Connection ~ 5700 5300
+Wire Wire Line
+	5700 5300 5700 5750
+Wire Wire Line
+	3150 4550 5700 4550
+Wire Wire Line
+	5700 2100 9000 2100
+Wire Wire Line
+	9000 2100 9000 5750
+Connection ~ 5700 2100
+Wire Wire Line
+	5700 2350 5700 3750
+Connection ~ 3150 4550
+Wire Wire Line
+	3150 4550 3150 6250
 $EndSCHEMATC
